File: dimmer-2ch.sch (KiCad schematic (older format))
At the start: 2 parts, among them J1 Conn_01x07, J2 Conn_01x04

Commit message: started layout
Parts:
- removed J2: Conn_01x04, Connector_Wire:SolderWirePad_1x04_P7.62mm_Drill2.5mm, symbol Connector_Generic:Conn_01x04
- added J2: Conn_01x03, Connector_Wire:SolderWirePad_1x03_P7.62mm_Drill2.5mm, symbol Connector_Generic:Conn_01x03
- added J3: Conn_01x03, Connector_PinHeader_2.54mm:PinHeader_1x03_P2.54mm_Vertical, symbol Connector_Generic:Conn_01x03
Connections:
- wire segments 28 -> 30
Changed lines of the file:
@@
 EESchema Schematic File Version 4
-EELAYER 29 0
+LIBS:dimmer-2ch-cache
+EELAYER 26 0
 EELAYER END
 $Descr A4 11693 8268
@@
 $EndDescr
 $Comp
-L Connector_Generic:Conn_01x04 J2
-U 1 1 5BF27495
-P 3525 4525
-F 0 "J2" H 3443 4100 50  0000 C CNN
-F 1 "Conn_01x04" H 3443 4191 50  0000 C CNN
-F 2 "Connector_Wire:SolderWirePad_1x04_P7.62mm_Drill2.5mm" H 3525 4525 50  0001 C CNN
-F 3 "~" H 3525 4525 50  0001 C CNN
-	1    3525 4525
-	-1   0    0    1
-$EndComp
-$Comp
 L power:GND #PWR0101
 U 1 1 5BF2A93F
-P 3750 3800
-F 0 "#PWR0101" H 3750 3550 50  0001 C CNN
-F 1 "GND" H 3825 3675 50  0000 C CNN
-F 2 "" H 3750 3800 50  0001 C CNN
-F 3 "" H 3750 3800 50  0001 C CNN
-	1    3750 3800
+P 4000 3050
+F 0 "#PWR0101" H 4000 2800 50  0001 C CNN
+F 1 "GND" H 4075 2925 50  0000 C CNN
+F 2 "" H 4000 3050 50  0001 C CNN
+F 3 "" H 4000 3050 50  0001 C CNN
+	1    4000 3050
 	1    0    0    -1
 $EndComp
 Wire Wire Line
-	3750 3800 3750 3775
-Wire Wire Line
-	3750 3775 3725 3775
-Text Label 3775 3675 0    50   ~ 0
-5V
-Wire Wire Line
-	3725 3675 3775 3675
-Text Label 6225 2875 2    50   ~ 0
-5V
-Wire Wire Line
-	6225 2875 6250 2875
-Text Label 6225 5450 2    50   ~ 0
-5V
-Wire Wire Line
-	6225 5450 6250 5450
-$Sheet
-S 6250 2800 725  400
+	4000 3050 4000 3025
+Wire Wire Line
+	4000 3025 3975 3025
+Text Label 4025 2925 0    50   ~ 0
+5V
+Wire Wire Line
+	3975 2925 4025 2925
+Text Label 6625 2425 2    50   ~ 0
+5V
+Wire Wire Line
+	6625 2425 6650 2425
+Text Label 5950 4775 2    50   ~ 0
+5V
+Wire Wire Line
+	5950 4775 5975 4775
+$Sheet
+S 6650 2350 725  400
 U 5BF2BC14
 F0 "current sense 1" 50
 F1 "current_sense.sch" 50
-F2 "IN" I L 6250 3075 50
-F3 "OUT" O R 6975 3075 50
-F4 "ANALOG_OUT" O R 6975 2875 50
-F5 "5V" I L 6250 2875 50
-$EndSheet
-$Sheet
-S 5150 2800 625  450
+F2 "IN" I L 6650 2625 50
+F3 "OUT" O R 7375 2625 50
+F4 "ANALOG_OUT" O R 7375 2425 50
+F5 "5V" I L 6650 2425 50
+$EndSheet
+$Sheet
+S 5550 2350 625  450
 U 5BF2C123
 F0 "triac 1" 50
 F1 "triac.sch" 50
-F2 "DIGITAL_IN" I L 5150 2900 50
-F3 "OUT" O R 5775 3075 50
-F4 "IN" I L 5150 3075 50
-$EndSheet
-Wire Wire Line
-	5775 3075 6250 3075
-Text Label 7000 3075 0    50   ~ 0
+F2 "DIGITAL_IN" I L 5550 2450 50
+F3 "OUT" O R 6175 2625 50
+F4 "IN" I L 5550 2625 50
+$EndSheet
+Wire Wire Line
+	6175 2625 6650 2625
+Text Label 7400 2625 0    50   ~ 0
 LINE_OUT_1
 Wire Wire Line
-	7000 3075 6975 3075
-Text Label 5125 3075 2    50   ~ 0
-LINE_IN
-Wire Wire Line
-	5125 3075 5150 3075
-Text Label 5125 2900 2    50   ~ 0
+	7400 2625 7375 2625
+Text Label 5525 2625 2    50   ~ 0
+LINE_IN
+Wire Wire Line
+	5525 2625 5550 2625
+Text Label 5525 2450 2    50   ~ 0
 TRIAC_1
 Wire Wire Line
-	5125 2900 5150 2900
-Text Label 7000 2875 0    50   ~ 0
+	5525 2450 5550 2450
+Text Label 7400 2425 0    50   ~ 0
 CURRENT_SENSE_1
 Wire Wire Line
-	7000 2875 6975 2875
-Text Label 3775 3475 0    50   ~ 0
+	7400 2425 7375 2425
+Text Label 4025 2725 0    50   ~ 0
 CURRENT_SENSE_1
 Wire Wire Line
-	3775 3275 3725 3275
-Text Label 3775 3275 0    50   ~ 0
+	4025 2525 3975 2525
+Text Label 4025 2525 0    50   ~ 0
 TRIAC_1
 Wire Wire Line
-	3775 3375 3725 3375
-Text Label 3775 3375 0    50   ~ 0
+	4025 2625 3975 2625
+Text Label 4025 2625 0    50   ~ 0
 TRIAC_2
 Wire Wire Line
-	3775 3475 3725 3475
-Text Label 3775 3575 0    50   ~ 0
+	4025 2725 3975 2725
+Text Label 4025 2825 0    50   ~ 0
 CURRENT_SENSE_2
 Wire Wire Line
-	3775 3575 3725 3575
-Text Label 3775 4425 0    50   ~ 0
-LINE_IN
-Wire Wire Line
-	3775 4525 3725 4525
-Text Label 3775 4625 0    50   ~ 0
+	4025 2825 3975 2825
+Text Label 4025 3825 0    50   ~ 0
+LINE_IN
+Wire Wire Line
+	4025 3925 3975 3925
+Text Label 4025 4500 0    50   ~ 0
 NEUTRAL
 Wire Wire Line
-	3775 4625 3725 4625
-$Sheet
-S 6250 5350 750  525
+	4025 4500 3975 4500
+$Sheet
+S 5975 4675 750  525
 U 5BF2E568
 F0 "zerocross" 50
 F1 "zerocross.sch" 50
-F2 "LINE" I L 6250 5675 50
-F3 "NEUTRAL" I L 6250 5750 50
-F4 "DIGITAL_OUT" O R 7000 5550 50
-F5 "5V" I L 6250 5450 50
-$EndSheet
-Text Label 6200 5675 2    50   ~ 0
-LINE_IN
-Wire Wire Line
-	6200 5675 6250 5675
-Text Label 6200 5750 2    50   ~ 0
+F2 "LINE" I L 5975 5000 50
+F3 "NEUTRAL" I L 5975 5075 50
+F4 "DIGITAL_OUT" O R 6725 4875 50
+F5 "5V" I L 5975 4775 50
+$EndSheet
+Text Label 5925 5000 2    50   ~ 0
+LINE_IN
+Wire Wire Line
+	5925 5000 5975 5000
+Text Label 5925 5075 2    50   ~ 0
 NEUTRAL
 Wire Wire Line
-	6200 5750 6250 5750
+	5925 5075 5975 5075
 $Comp
 L Connector_Generic:Conn_01x07 J1
 U 1 1 5BF2F7D8
-P 3525 3475
-F 0 "J1" H 3443 2950 50  0000 C CNN
-F 1 "Conn_01x07" H 3443 3041 50  0000 C CNN
-F 2 "Connector_PinHeader_2.54mm:PinHeader_1x07_P2.54mm_Vertical" H 3525 3475 50  0001 C CNN
-F 3 "~" H 3525 3475 50  0001 C CNN
-	1    3525 3475
+P 3775 2725
+F 0 "J1" H 3693 2200 50  0000 C CNN
+F 1 "Conn_01x07" H 3693 2291 50  0000 C CNN
+F 2 "Connector_PinHeader_2.54mm:PinHeader_1x07_P2.54mm_Vertical" H 3775 2725 50  0001 C CNN
+F 3 "~" H 3775 2725 50  0001 C CNN
+	1    3775 2725
 	-1   0    0    1
 $EndComp
-Text Label 3775 3175 0    50   ~ 0
+Text Label 4025 2425 0    50   ~ 0
 ZEROCROSS
 Wire Wire Line
-	3775 3175 3725 3175
-Text Label 7025 5550 0    50   ~ 0
+	4025 2425 3975 2425
+Text Label 6750 4875 0    50   ~ 0
 ZEROCROSS
 Wire Wire Line
-	7025 5550 7000 5550
-Text Label 6225 4000 2    50   ~ 0
-5V
-Wire Wire Line
-	6225 4000 6250 4000
-$Sheet
-S 6250 3925 725  400
+	6750 4875 6725 4875
+Text Label 6625 3550 2    50   ~ 0
+5V
+Wire Wire Line
+	6625 3550 6650 3550
+$Sheet
+S 6650 3475 725  400
 U 5BF337E0
 F0 "current sense 2" 50
 F1 "current_sense.sch" 50
-F2 "IN" I L 6250 4200 50
-F3 "OUT" O R 6975 4200 50
-F4 "ANALOG_OUT" O R 6975 4000 50
-F5 "5V" I L 6250 4000 50
-$EndSheet
-$Sheet
-S 5150 3925 625  450
+F2 "IN" I L 6650 3750 50
+F3 "OUT" O R 7375 3750 50
+F4 "ANALOG_OUT" O R 7375 3550 50
+F5 "5V" I L 6650 3550 50
+$EndSheet
+$Sheet
+S 5550 3475 625  450
 U 5BF337E5
 F0 "triac 2" 50
 F1 "triac.sch" 50
-F2 "DIGITAL_IN" I L 5150 4025 50
-F3 "OUT" O R 5775 4200 50
-F4 "IN" I L 5150 4200 50
-$EndSheet
-Wire Wire Line
-	5775 4200 6250 4200
-Text Label 7000 4200 0    50   ~ 0
+F2 "DIGITAL_IN" I L 5550 3575 50
+F3 "OUT" O R 6175 3750 50
+F4 "IN" I L 5550 3750 50
+$EndSheet
+Wire Wire Line
+	6175 3750 6650 3750
+Text Label 7400 3750 0    50   ~ 0
 LINE_OUT_2
 Wire Wire Line
-	7000 4200 6975 4200
-Text Label 5125 4200 2    50   ~ 0
-LINE_IN
-Wire Wire Line
-	5125 4200 5150 4200
-Text Label 5125 4025 2    50   ~ 0
+	7400 3750 7375 3750
+Text Label 5525 3750 2    50   ~ 0
+LINE_IN
+Wire Wire Line
+	5525 3750 5550 3750
+Text Label 5525 3575 2    50   ~ 0
 TRIAC_1
 Wire Wire Line
-	5125 4025 5150 4025
-Text Label 7000 4000 0    50   ~ 0
+	5525 3575 5550 3575
+Text Label 7400 3550 0    50   ~ 0
 CURRENT_SENSE_1
 Wire Wire Line
-	7000 4000 6975 4000
-Text Label 3775 4325 0    50   ~ 0
+	7400 3550 7375 3550
+Text Label 4025 3725 0    50   ~ 0
 LINE_OUT_1
 Wire Wire Line
-	3775 4325 3725 4325
-Wire Wire Line
-	3775 4425 3725 4425
-Text Label 3775 4525 0    50   ~ 0
+	4025 3725 3975 3725
+Wire Wire Line
+	4025 3825 3975 3825
+Text Label 4025 3925 0    50   ~ 0
 LINE_OUT_2
+$Comp
+L Connector_Generic:Conn_01x03 J2
+U 1 1 5BF0CB92
+P 3775 3825
+F 0 "J2" H 3695 3500 50  0000 C CNN
+F 1 "Conn_01x03" H 3695 3591 50  0000 C CNN
+F 2 "Connector_Wire:SolderWirePad_1x03_P7.62mm_Drill2.5mm" H 3775 3825 50  0001 C CNN
+F 3 "~" H 3775 3825 50  0001 C CNN
+	1    3775 3825
+	-1   0    0    1
+$EndComp
+Text Label 4025 4400 0    50   ~ 0
+LINE_IN
+Wire Wire Line
+	4025 4400 3975 4400
+$Comp
+L Connector_Generic:Conn_01x03 J3
+U 1 1 5BF108AF
+P 3775 4500
+F 0 "J3" H 3695 4175 50  0000 C CNN
+F 1 "Conn_01x03" H 3695 4266 50  0000 C CNN
+F 2 "Connector_PinHeader_2.54mm:PinHeader_1x03_P2.54mm_Vertical" H 3775 4500 50  0001 C CNN
+F 3 "~" H 3775 4500 50  0001 C CNN
+	1    3775 4500
+	-1   0    0    1
+$EndComp
+Text Label 4025 4600 0    50   ~ 0
+NEUTRAL
+Wire Wire Line
+	4025 4600 3975 4600
 $EndSCHEMATC

Commit message: finished layout, final check
Parts:
- removed J1: Conn_01x07, Connector_PinHeader_2.54mm:PinHeader_1x07_P2.54mm_Vertical, symbol Connector_Generic:Conn_01x07
- added J1: Conn_01x04, Connector_PinHeader_2.54mm:PinHeader_1x04_P2.54mm_Vertical, symbol Connector_Generic:Conn_01x04
- added J4: Conn_01x05, Connector_PinHeader_2.54mm:PinHeader_1x05_P2.54mm_Vertical, symbol Connector_Generic:Conn_01x05
- J2, J3: symbol Connector_Generic:Conn_01x03 -> dimmer-2ch-rescue:Conn_01x03-Connector_Generic
Connections:
- wire segments 30 -> 31
Changed lines of the file:
@@
 Comment4 ""
 $EndDescr
-$Comp
-L power:GND #PWR0101
-U 1 1 5BF2A93F
-P 4000 3050
-F 0 "#PWR0101" H 4000 2800 50  0001 C CNN
-F 1 "GND" H 4075 2925 50  0000 C CNN
-F 2 "" H 4000 3050 50  0001 C CNN
-F 3 "" H 4000 3050 50  0001 C CNN
-	1    4000 3050
-	1    0    0    -1
-$EndComp
-Wire Wire Line
-	4000 3050 4000 3025
-Wire Wire Line
-	4000 3025 3975 3025
-Text Label 4025 2925 0    50   ~ 0
-5V
-Wire Wire Line
-	3975 2925 4025 2925
-Text Label 6625 2425 2    50   ~ 0
-5V
-Wire Wire Line
-	6625 2425 6650 2425
+Text Label 6800 2450 2    50   ~ 0
+5V
+Wire Wire Line
+	6800 2450 6825 2450
 Text Label 5950 4775 2    50   ~ 0
 5V
@@
 	5950 4775 5975 4775
 $Sheet
-S 6650 2350 725  400
+S 6825 2375 725  400
 U 5BF2BC14
 F0 "current sense 1" 50
 F1 "current_sense.sch" 50
-F2 "IN" I L 6650 2625 50
-F3 "OUT" O R 7375 2625 50
-F4 "ANALOG_OUT" O R 7375 2425 50
-F5 "5V" I L 6650 2425 50
-$EndSheet
-$Sheet
-S 5550 2350 625  450
+F2 "IN" I L 6825 2650 50
+F3 "OUT" O R 7550 2650 50
+F4 "ANALOG_OUT" O R 7550 2450 50
+F5 "5V" I L 6825 2450 50
+$EndSheet
+$Sheet
+S 5700 2375 625  450
 U 5BF2C123
 F0 "triac 1" 50
 F1 "triac.sch" 50
-F2 "DIGITAL_IN" I L 5550 2450 50
-F3 "OUT" O R 6175 2625 50
-F4 "IN" I L 5550 2625 50
-$EndSheet
-Wire Wire Line
-	6175 2625 6650 2625
-Text Label 7400 2625 0    50   ~ 0
+F2 "DIGITAL_IN" I L 5700 2475 50
+F3 "OUT" O R 6325 2650 50
+F4 "IN" I L 5700 2650 50
+$EndSheet
+Text Label 7575 2650 0    50   ~ 0
 LINE_OUT_1
-Wire Wire Line
-	7400 2625 7375 2625
-Text Label 5525 2625 2    50   ~ 0
-LINE_IN
-Wire Wire Line
-	5525 2625 5550 2625
-Text Label 5525 2450 2    50   ~ 0
+Text Label 5675 2650 2    50   ~ 0
+LINE_IN
+Text Label 5675 2475 2    50   ~ 0
 TRIAC_1
 Wire Wire Line
-	5525 2450 5550 2450
-Text Label 7400 2425 0    50   ~ 0
+	5675 2475 5700 2475
+Text Label 7575 2450 0    50   ~ 0
 CURRENT_SENSE_1
 Wire Wire Line
-	7400 2425 7375 2425
+	7575 2450 7550 2450
 Text Label 4025 2725 0    50   ~ 0
 CURRENT_SENSE_1
@@
 Wire Wire Line
 	5925 5075 5975 5075
-$Comp
-L Connector_Generic:Conn_01x07 J1
-U 1 1 5BF2F7D8
-P 3775 2725
-F 0 "J1" H 3693 2200 50  0000 C CNN
-F 1 "Conn_01x07" H 3693 2291 50  0000 C CNN
-F 2 "Connector_PinHeader_2.54mm:PinHeader_1x07_P2.54mm_Vertical" H 3775 2725 50  0001 C CNN
-F 3 "~" H 3775 2725 50  0001 C CNN
-	1    3775 2725
-	-1   0    0    1
-$EndComp
 Text Label 4025 2425 0    50   ~ 0
 ZEROCROSS
@@
 Wire Wire Line
 	6750 4875 6725 4875
-Text Label 6625 3550 2    50   ~ 0
-5V
-Wire Wire Line
-	6625 3550 6650 3550
-$Sheet
-S 6650 3475 725  400
+Text Label 6750 3575 2    50   ~ 0
+5V
+Wire Wire Line
+	6750 3575 6775 3575
+$Sheet
+S 6775 3500 725  400
 U 5BF337E0
 F0 "current sense 2" 50
 F1 "current_sense.sch" 50
-F2 "IN" I L 6650 3750 50
-F3 "OUT" O R 7375 3750 50
-F4 "ANALOG_OUT" O R 7375 3550 50
-F5 "5V" I L 6650 3550 50
-$EndSheet
-$Sheet
-S 5550 3475 625  450
+F2 "IN" I L 6775 3775 50
+F3 "OUT" O R 7500 3775 50
+F4 "ANALOG_OUT" O R 7500 3575 50
+F5 "5V" I L 6775 3575 50
+$EndSheet
+$Sheet
+S 5725 3500 625  450
 U 5BF337E5
 F0 "triac 2" 50
 F1 "triac.sch" 50
-F2 "DIGITAL_IN" I L 5550 3575 50
-F3 "OUT" O R 6175 3750 50
-F4 "IN" I L 5550 3750 50
-$EndSheet
-Wire Wire Line
-	6175 3750 6650 3750
-Text Label 7400 3750 0    50   ~ 0
+F2 "DIGITAL_IN" I L 5725 3600 50
+F3 "OUT" O R 6350 3775 50
+F4 "IN" I L 5725 3775 50
+$EndSheet
+Text Label 7525 3775 0    50   ~ 0
 LINE_OUT_2
-Wire Wire Line
-	7400 3750 7375 3750
-Text Label 5525 3750 2    50   ~ 0
-LINE_IN
-Wire Wire Line
-	5525 3750 5550 3750
-Text Label 5525 3575 2    50   ~ 0
-TRIAC_1
-Wire Wire Line
-	5525 3575 5550 3575
-Text Label 7400 3550 0    50   ~ 0
-CURRENT_SENSE_1
-Wire Wire Line
-	7400 3550 7375 3550
+Text Label 5700 3775 2    50   ~ 0
+LINE_IN
+Text Label 5700 3600 2    50   ~ 0
+TRIAC_2
+Wire Wire Line
+	5700 3600 5725 3600
+Text Label 7525 3575 0    50   ~ 0
+CURRENT_SENSE_2
+Wire Wire Line
+	7525 3575 7500 3575
 Text Label 4025 3725 0    50   ~ 0
 LINE_OUT_1
@@
 LINE_OUT_2
 $Comp
-L Connector_Generic:Conn_01x03 J2
+L dimmer-2ch-rescue:Conn_01x03-Connector_Generic J2
 U 1 1 5BF0CB92
 P 3775 3825
@@
 	4025 4400 3975 4400
 $Comp
-L Connector_Generic:Conn_01x03 J3
+L dimmer-2ch-rescue:Conn_01x03-Connector_Generic J3
 U 1 1 5BF108AF
 P 3775 4500
@@
 Wire Wire Line
 	4025 4600 3975 4600
+$Comp
+L Connector_Generic:Conn_01x04 J1
+U 1 1 5BF18045
+P 2625 3800
+F 0 "J1" H 2545 3375 50  0000 C CNN
+F 1 "Conn_01x04" H 2545 3466 50  0000 C CNN
+F 2 "Connector_PinHeader_2.54mm:PinHeader_1x04_P2.54mm_Vertical" H 2625 3800 50  0001 C CNN
+F 3 "~" H 2625 3800 50  0001 C CNN
+	1    2625 3800
+	-1   0    0    1
+$EndComp
+$Comp
+L dimmer-2ch-rescue:GND-power #PWR0101
+U 1 1 5BF1810D
+P 2875 3900
+F 0 "#PWR0101" H 2875 3650 50  0001 C CNN
+F 1 "GND" V 2825 3750 50  0000 C CNN
+F 2 "" H 2875 3900 50  0001 C CNN
+F 3 "" H 2875 3900 50  0001 C CNN
+	1    2875 3900
+	0    -1   -1   0
+$EndComp
+$Comp
+L dimmer-2ch-rescue:GND-power #PWR0110
+U 1 1 5BF1891F
+P 2875 3800
+F 0 "#PWR0110" H 2875 3550 50  0001 C CNN
+F 1 "GND" V 2825 3650 50  0000 C CNN
+F 2 "" H 2875 3800 50  0001 C CNN
+F 3 "" H 2875 3800 50  0001 C CNN
+	1    2875 3800
+	0    -1   -1   0
+$EndComp
+Wire Wire Line
+	2825 3800 2875 3800
+Wire Wire Line
+	2825 3900 2875 3900
+Text Label 2900 3600 0    50   ~ 0
+5V
+Wire Wire Line
+	2900 3600 2825 3600
+Text Label 2900 3700 0    50   ~ 0
+5V
+Wire Wire Line
+	2900 3700 2825 3700
+$Comp
+L Connector_Generic:Conn_01x05 J4
+U 1 1 5BF1B073
+P 3775 2625
+F 0 "J4" H 3695 2200 50  0000 C CNN
+F 1 "Conn_01x05" H 3695 2291 50  0000 C CNN
+F 2 "Connector_PinHeader_2.54mm:PinHeader_1x05_P2.54mm_Vertical" H 3775 2625 50  0001 C CNN
+F 3 "~" H 3775 2625 50  0001 C CNN
+	1    3775 2625
+	-1   0    0    1
+$EndComp
+Wire Wire Line
+	5675 2650 5700 2650
+Wire Wire Line
+	5700 3775 5725 3775
+Wire Wire Line
+	7525 3775 7500 3775
+Wire Wire Line
+	7575 2650 7550 2650
+Wire Wire Line
+	6325 2650 6825 2650
+Wire Wire Line
+	6350 3775 6775 3775
 $EndSCHEMATC
