File: zerocross.sch (KiCad schematic (older format))
At the start: 6 parts, among them U3 H11AA1

Commit message: started layout
Parts:
- R5, R6, R7, R8, R9: symbol open-automation:R_10k -> dimmer-2ch-rescue:R_10k-open-automation
- U3: symbol open-automation:H11AA1 -> dimmer-2ch-rescue:H11AA1-open-automation
Changed lines of the file:
@@
 EESchema Schematic File Version 4
-EELAYER 29 0
+LIBS:dimmer-2ch-cache
+EELAYER 26 0
 EELAYER END
 $Descr A4 11693 8268
@@
 $EndDescr
 $Comp
-L open-automation:R_10k R?
+L dimmer-2ch-rescue:R_10k-open-automation R?
 U 1 1 5BF1128B
 P 6925 2925
@@
 $EndComp
 $Comp
-L open-automation:H11AA1 U?
+L dimmer-2ch-rescue:H11AA1-open-automation U?
 U 1 1 5BF18D83
 P 7475 3025
@@
 	7175 2925 7075 2925
 $Comp
-L open-automation:R_10k R?
+L dimmer-2ch-rescue:R_10k-open-automation R?
 U 1 1 5BF1A86E
 P 6925 3125
@@
 	7800 3125 7775 3125
 $Comp
-L open-automation:R_10k R?
+L dimmer-2ch-rescue:R_10k-open-automation R?
 U 1 1 5BF1BEB8
 P 7825 2725
@@
 Connection ~ 7825 2925
 $Comp
-L open-automation:R_10k R?
+L dimmer-2ch-rescue:R_10k-open-automation R?
 U 1 1 5BF1D45B
 P 8400 2000
@@
 $EndComp
 $Comp
-L open-automation:R_10k R?
+L dimmer-2ch-rescue:R_10k-open-automation R?
 U 1 1 5BF1EB6A
 P 8400 2350

Commit message: finished layout, final check
Changed lines of the file:
@@
 	6775 3125 6725 3125
 $Comp
-L power:GND #PWR?
+L dimmer-2ch-rescue:GND-power #PWR?
 U 1 1 5BF1B461
 P 7800 3150
@@
 $EndComp
 $Comp
-L power:GND #PWR?
+L dimmer-2ch-rescue:GND-power #PWR?
 U 1 1 5BF1F20C
 P 8400 2550
