File: dimmer-2ch.kicad_pcb (KiCad board)
At the start: 2 copper layers, 26 parts, among them J1 Conn_01x07, J2 Conn_01x04, U1 ACS712xLCTR-30A, U2 MOC3052M, U3 H11AA1, U4 ACS712xLCTR-30A, U5 MOC3052M

Commit message: started layout
Parts:
- added J3: Conn_01x03, Connector_PinHeader_2.54mm:PinHeader_1x03_P2.54mm_Vertical, F.Cu at (205.2, 31.8)
- J2: value Conn_01x04 -> Conn_01x03; footprint Connector_Wire:SolderWirePad_1x04_P7.62mm_Drill2.5mm -> Connector_Wire:SolderWirePad_1x03_P7.62mm_Drill2.5mm
- moved R5 73.4 mm to (201.9, 36.6), turned to 270 degrees
- moved R6 72.2 mm to (201.9, 32.5), turned to 90 degrees
- moved R2 65.5 mm to (176.4, 78.0), turned to 180 degrees
- moved C1 58.7 mm to (190.0, 75.9), turned to 90 degrees
- moved U5 47.2 mm to (173.9, 53.3)
- moved R7 46.7 mm to (153.9, 62.3)
- moved R8 46.7 mm to (153.9, 64.8)
- moved R9 46.7 mm to (158.2, 62.3)
- moved R13 42.6 mm to (164.1, 69.2)
- moved R4 42.6 mm to (164.1, 61.0)
- moved R12 40.5 mm to (176.2, 46.0), turned to 180 degrees
- moved R3 39.1 mm to (171.4, 78.0), turned to 180 degrees
- moved R1 37.3 mm to (176.3, 63.2), turned to 180 degrees
- moved R10 32.7 mm to (171.4, 60.2)
- moved R11 31.1 mm to (171.8, 46.0), turned to 180 degrees
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Connections:
- J2 pad 1: /NEUTRAL -> /LINE_OUT_2
- J2 pad 2: /LINE_OUT_2 -> /LINE_IN
- J2 pad 3: /LINE_IN -> /LINE_OUT_1

Commit message: finished layout, final check
Parts:
- added J4: Conn_01x05, Connector_PinHeader_2.54mm:PinHeader_1x05_P2.54mm_Vertical, F.Cu at (121.4, 91.9)
- J1: value Conn_01x07 -> Conn_01x04; footprint Connector_PinHeader_2.54mm:PinHeader_1x07_P2.54mm_Vertical -> Connector_PinHeader_2.54mm:PinHeader_1x04_P2.54mm_Vertical
- moved U3 93.0 mm to (131.4, 105.0), turned to 270 degrees
- moved J3 88.5 mm to (136.1, 86.9), turned to 90 degrees
- moved R6 88.0 mm to (135.2, 89.9), turned to 0 degrees
- moved R5 81.5 mm to (140.5, 90.0), turned to 0 degrees
- moved C3 66.5 mm to (156.3, 99.1)
- moved U4 65.8 mm to (161.5, 99.3)
- moved R12 63.6 mm to (148.3, 103.1)
- moved R9 59.6 mm to (130.9, 115.3)
- moved R1 58.3 mm to (139.3, 108.3)
- moved J1 58.1 mm to (121.5, 106.7)
- moved D1 57.4 mm to (160.5, 115.8), turned to 180 degrees
- moved R8 57.1 mm to (130.9, 117.1), turned to 180 degrees
- moved R7 56.1 mm to (130.9, 113.5), turned to 180 degrees
- moved C2 54.7 mm to (166.6, 107.8), turned to 270 degrees
- moved U5 53.5 mm to (144.1, 97.8), turned to 0 degrees
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Connections:
- J1 pad 2: /5V -> GND
- J1 pad 3: /CURRENT_SENSE_2 -> /5V
- J1 pad 4: /CURRENT_SENSE_1 -> /5V
- R10 pad 2: /TRIAC_1 -> /TRIAC_2
- U4 pad 7: /CURRENT_SENSE_1 -> /CURRENT_SENSE_2
Routing:
- net /5V: track 0.00 -> 63.7 mm, vias 0 -> 2
- net /LINE_IN: track 0.00 -> 49.9 mm
- net /CURRENT_SENSE_2: track 0.00 -> 48.7 mm
- net /CURRENT_SENSE_1: track 0.00 -> 45.9 mm, vias 0 -> 2
- net GND: track 0.00 -> 42.5 mm, vias 0 -> 6
- net Net-(D2-Pad3): track 0.00 -> 29.4 mm, vias 0 -> 2
- net Net-(D1-Pad3): track 0.00 -> 23.2 mm, vias 0 -> 2
- net /current sense 2/IN: track 0.00 -> 22.7 mm, vias 0 -> 5
- net /current sense 1/IN: track 0.00 -> 20.8 mm, vias 0 -> 5
- net /TRIAC_1: track 0.00 -> 20.6 mm
- net /TRIAC_2: track 0.00 -> 19.4 mm, vias 0 -> 1
- net /ZEROCROSS: track 0.00 -> 18.3 mm
- net Net-(R5-Pad1): track 0.00 -> 15.4 mm
- net /LINE_OUT_1: track 0.00 -> 14.7 mm
- net /LINE_OUT_2: track 0.00 -> 13.4 mm
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- added copper zone on F.Cu, net /LINE_IN
- added copper zone on B.Cu, net /current sense 1/IN
- added copper zone on B.Cu, net /current sense 2/IN
- added copper zone on B.Cu, net GND
Other:
- board outline added: 61.7 x 40.6 mm
- net class HIGH POWER added: clearance 0.4, trace_width 1.5, via_dia 2, via_drill 1
- board text added: "5V"
- board text added: "CS1"
- board text added: "CS2"
- board text added: "GND"
- board text added: "LINE IN"
- board text added: "LINE_OUT_1"
- board text added: "LINE_OUT_2"
- board text added: "NEUTRAL"
- board text added: "T1"
- board text added: "T2"
- board text added: "ZC"

Commit message: increased clearences
Routing:
- net /current sense 1/IN: track 20.8 -> 31.1 mm
- net /current sense 2/IN: track 22.7 -> 27.9 mm

Commit message: ready for board house
Parts:
- added LOGO: , open-automation:LOGO, B.Cu at (153.4, 117.7)
Other:
- board text added: "Dimmer v0.0.1"
