File: triac.sch (KiCad schematic (older format))
At the start: 7 parts, among them U2 MOC3052M

Commit message: started layout
Parts:
- C2: symbol open-automation:C_0.1uF -> dimmer-2ch-rescue:C_0.1uF-open-automation
- R1, R3: symbol open-automation:R_470 -> dimmer-2ch-rescue:R_470-open-automation
- R2, R4: symbol open-automation:R_27 -> dimmer-2ch-rescue:R_27-open-automation
Changed lines of the file:
@@
 EESchema Schematic File Version 4
-EELAYER 29 0
+LIBS:dimmer-2ch-cache
+EELAYER 26 0
 EELAYER END
 $Descr A4 11693 8268
 encoding utf-8
-Sheet 6 6
+Sheet 3 6
 Title ""
 Date ""
@@
 AR Path="/5BF2C123/5BEFC71E" Ref="U2"  Part="1"
 AR Path="/5BF337E5/5BEFC71E" Ref="U5"  Part="1"
-F 0 "U5" H 4725 3675 50  0000 C CNN
+F 0 "U2" H 4725 3675 50  0000 C CNN
 F 1 "MOC3052M" H 4725 3584 50  0000 C CNN
 F 2 "Package_DIP:SMDIP-6_W9.53mm_Clearance8mm" H 4525 3150 50  0001 L CIN
@@
 $EndComp
 $Comp
-L open-automation:R_470 R?
+L dimmer-2ch-rescue:R_470-open-automation R?
 U 1 1 5BEFC725
 P 4225 3250
@@
 AR Path="/5BF2C123/5BEFC725" Ref="R1"  Part="1"
 AR Path="/5BF337E5/5BEFC725" Ref="R10"  Part="1"
-F 0 "R10" V 4225 3200 50  0000 L CNN
+F 0 "R1" V 4225 3200 50  0000 L CNN
 F 1 "R_470" V 4125 3125 50  0000 L CNN
 F 2 "Resistor_SMD:R_0603_1608Metric_Pad1.05x0.95mm_HandSolder" V 4155 3250 50  0001 C CNN
@@
 AR Path="/5BF2C123/5BEFC72B" Ref="#PWR0104"  Part="1"
 AR Path="/5BF337E5/5BEFC72B" Ref="#PWR0109"  Part="1"
-F 0 "#PWR0109" H 4400 3225 50  0001 C CNN
+F 0 "#PWR0104" H 4400 3225 50  0001 C CNN
 F 1 "GND" H 4405 3302 50  0000 C CNN
 F 2 "" H 4400 3475 50  0001 C CNN
@@
 AR Path="/5BF2C123/5BF04A14" Ref="D1"  Part="1"
 AR Path="/5BF337E5/5BF04A14" Ref="D2"  Part="1"
-F 0 "D2" H 5803 3396 50  0000 L CNN
+F 0 "D1" H 5803 3396 50  0000 L CNN
 F 1 "Q_TRIAC_A1A2G" H 5803 3305 50  0000 L CNN
 F 2 "Package_TO_SOT_SMD:TO-263-2" V 5750 3375 50  0001 C CNN
@@
 $EndComp
 $Comp
-L open-automation:R_470 R?
+L dimmer-2ch-rescue:R_470-open-automation R?
 U 1 1 5BF05572
 P 5375 3550
@@
 AR Path="/5BF2C123/5BF05572" Ref="R3"  Part="1"
 AR Path="/5BF337E5/5BF05572" Ref="R12"  Part="1"
-F 0 "R12" V 5375 3500 50  0000 L CNN
+F 0 "R3" V 5375 3500 50  0000 L CNN
 F 1 "R_470" V 5475 3450 50  0000 L CNN
 F 2 "Resistor_SMD:R_0603_1608Metric_Pad1.05x0.95mm_HandSolder" V 5305 3550 50  0001 C CNN
@@
 	5100 3250 5100 3150
 $Comp
-L open-automation:R_27 R?
+L dimmer-2ch-rescue:R_27-open-automation R?
 U 1 1 5BF077A1
 P 6850 3225
@@
 AR Path="/5BF2C123/5BF077A1" Ref="R4"  Part="1"
 AR Path="/5BF337E5/5BF077A1" Ref="R13"  Part="1"
-F 0 "R13" H 6900 3250 50  0000 L CNN
+F 0 "R4" H 6900 3250 50  0000 L CNN
 F 1 "R_27" H 6900 3175 50  0000 L CNN
 F 2 "Resistor_SMD:R_0603_1608Metric_Pad1.05x0.95mm_HandSolder" V 6780 3225 50  0001 C CNN
@@
 $EndComp
 $Comp
-L open-automation:C_0.1uF C?
+L dimmer-2ch-rescue:C_0.1uF-open-automation C?
 U 1 1 5BF07CE5
 P 6850 3550
@@
 AR Path="/5BF2C123/5BF07CE5" Ref="C2"  Part="1"
 AR Path="/5BF337E5/5BF07CE5" Ref="C4"  Part="1"
-F 0 "C4" H 6950 3550 50  0000 L CNN
+F 0 "C2" H 6950 3550 50  0000 L CNN
 F 1 "C_0.1uF" H 6875 3450 50  0000 L CNN
 F 2 "Capacitor_SMD:C_0603_1608Metric_Pad1.05x0.95mm_HandSolder" H 6950 3850 50  0001 C CNN
@@
 	5175 3450 5525 3450
 $Comp
-L open-automation:R_27 R?
+L dimmer-2ch-rescue:R_27-open-automation R?
 U 1 1 5BF0B71E
 P 5375 3150
@@
 AR Path="/5BF2C123/5BF0B71E" Ref="R2"  Part="1"
 AR Path="/5BF337E5/5BF0B71E" Ref="R11"  Part="1"
-F 0 "R11" V 5375 3100 50  0000 L CNN
+F 0 "R2" V 5375 3100 50  0000 L CNN
 F 1 "R_27" V 5300 3050 50  0000 L CNN
 F 2 "Resistor_SMD:R_0603_1608Metric_Pad1.05x0.95mm_HandSolder" V 5305 3150 50  0001 C CNN

Commit message: finished layout, final check
Parts:
- D1: symbol Device:Q_TRIAC_A1A2G -> dimmer-2ch-rescue:Q_TRIAC_A1A2G-Device
- U2: symbol Relay_SolidState:MOC3052M -> dimmer-2ch-rescue:MOC3052M-Relay_SolidState
Changed lines of the file:
@@
 $EndDescr
 $Comp
-L Relay_SolidState:MOC3052M U?
+L dimmer-2ch-rescue:MOC3052M-Relay_SolidState U?
 U 1 1 5BEFC71E
 P 4725 3350
@@
 $EndComp
 $Comp
-L power:GND #PWR?
+L dimmer-2ch-rescue:GND-power #PWR?
 U 1 1 5BEFC72B
 P 4400 3475
@@
 AR Path="/5BF2C123/5BEFC72B" Ref="#PWR0104"  Part="1"
 AR Path="/5BF337E5/5BEFC72B" Ref="#PWR0109"  Part="1"
-F 0 "#PWR0104" H 4400 3225 50  0001 C CNN
+F 0 "#PWR0109" H 4400 3225 50  0001 C CNN
 F 1 "GND" H 4405 3302 50  0000 C CNN
 F 2 "" H 4400 3475 50  0001 C CNN
@@
 	4025 3250 4075 3250
 $Comp
-L Device:Q_TRIAC_A1A2G D?
+L dimmer-2ch-rescue:Q_TRIAC_A1A2G-Device D?
 U 1 1 5BF04A14
 P 5675 3350

Commit message: ready for board house
Parts:
- R2, R4: Part Number ERJ-3GEYJ2R2V -> ERJ-3GEYJ270V
Changed lines of the file:
@@
 F 2 "Resistor_SMD:R_0603_1608Metric_Pad1.05x0.95mm_HandSolder" V 6780 3225 50  0001 C CNN
 F 3 "https://www.digikey.com/product-detail/en/panasonic-electronic-components/ERJ-3GEYJ2R2V/P2.2GCT-ND/282413" V 6930 3225 50  0001 C CNN
-F 4 "ERJ-3GEYJ2R2V" V 7030 3325 60  0001 C CNN "Part Number"
+F 4 "ERJ-3GEYJ270V" V 7030 3325 60  0001 C CNN "Part Number"
 	1    6850 3225
 	1    0    0    -1
@@
 F 2 "Resistor_SMD:R_0603_1608Metric_Pad1.05x0.95mm_HandSolder" V 5305 3150 50  0001 C CNN
 F 3 "https://www.digikey.com/product-detail/en/panasonic-electronic-components/ERJ-3GEYJ2R2V/P2.2GCT-ND/282413" V 5455 3150 50  0001 C CNN
-F 4 "ERJ-3GEYJ2R2V" V 5555 3250 60  0001 C CNN "Part Number"
+F 4 "ERJ-3GEYJ270V" V 5555 3250 60  0001 C CNN "Part Number"
 	1    5375 3150
 	0    1    1    0
